Commit message: Implemented RGBD camera
	- Created URDF for RGBD and set up the sensor in gazebo simulation.
	- The camera feature remains but commented out.

File: description/depth_camera.xacro (robot description, xacro)
@@ -1,5 +1,5 @@
 <?xml version="1.0"?>
 <robot xmlns:xacro="http://www.ros.org/wiki/xacro" name="robot">
-    <!-- Camera -->
+    <!-- RGB_Depth camera -->
     <joint name="camera_joint" type="fixed">
         <parent link="chasis"/>
@@ -10,5 +10,5 @@
         <visual>
             <geometry>
-                <box size="0.01 0.03 0.03" />
+                <box size="0.01 0.09 0.03" />
             </geometry>
             <material name="orange"/>
@@ -21,15 +21,16 @@
     </joint>
     <link name="camera_link_optical"></link>
-    <!-- Camera in gazebo-->
+    <!-- RGBD camera in gazebo-->
     <gazebo reference="camera_link">
-        <sensor name="camera" type="camera">
-            <gz_frame_id>camera_link_optical</gz_frame_id>
+        <sensor name="camera" type="rgbd_camera">
+            <gz_frame_id>camera_link</gz_frame_id>
+            <frame_id>camera_link_optical</frame_id>
             <pose>0 0 0 0 0 0</pose>
-            <topic>camera/image_raw</topic>
-            <update_rate>30</update_rate>
+            <topic>camera/depth/image_raw</topic>
+            <update_rate>10</update_rate>
             <always_on>1</always_on>
             <visualize>true</visualize>
             <camera>
-                <horizontal_fov>1.089</horizontal_fov>
+                <horizontal_fov>2.0944</horizontal_fov>
                 <image>
                     <format>R8G8B8</format>
@@ -39,5 +40,5 @@
                 <clip>
                     <near>0.05</near>
-                    <far>8.0</far>
+                    <far>12.0</far>
                 </clip>
                 <!-- <distortion>

File: description/robot.urdf.xacro (robot description, xacro)
@@ -4,4 +4,5 @@
     <xacro:include filename = "gazebo_control.xacro" />
     <xacro:include filename = "lidar.xacro" />
-    <xacro:include filename = "camera.xacro" />
+    <!-- <xacro:include filename = "camera.xacro" /> -->
+    <xacro:include filename = "depth_camera.xacro" />
 </robot>
