Commit message: Implemented gz_ros2_control for differential drive. Implemented a basic velocity_publisher for the controller. Merge robot state publisher node into the sim.launch.py. deactivated gazebo_control (script still included but commented out).

File: description/gz_diff_drive_control.xacro (robot description, xacro)
@@ -16,5 +16,5 @@
             <odom_topic>odom</odom_topic>
             <odometry_source>world</odometry_source>
-            <odom_publish_frequency>50</odom_publish_frequency>
+            <odom_publish_frequency>30</odom_publish_frequency>
             <tf_topic>tf</tf_topic>
             <!-- Frames -->

File: description/robot.urdf.xacro (robot description, xacro)
@@ -1,6 +1,15 @@
 <?xml version="1.0"?>
 <robot xmlns:xacro="http://www.ros.org/wiki/xacro"  name="robot">
+    <xacro:arg name="use_ros2_control"              default="true"/>
+    <!-- Robot_frames -->
     <xacro:include filename = "robot_main.xacro" />
-    <xacro:include filename = "gazebo_control.xacro" />
+    <!-- Controls -->
+    <xacro:if value="$(arg use_ros2_control)">
+        <xacro:include filename = "ros2_control.xacro" />
+    </xacro:if>
+    <xacro:unless value="$(arg use_ros2_control)">
+        <xacro:include filename = "gz_diff_drive_control.xacro" />
+    </xacro:unless>
+    <!-- Sensors -->
     <xacro:include filename = "lidar.xacro" />
     <!-- <xacro:include filename = "camera.xacro" /> -->

File: description/robot_main.xacro (robot description, xacro)
@@ -65,5 +65,5 @@
         <collision>
             <geometry>
-                <cylinder radius = "0.05" length= "0.04"/>
+                <sphere radius = "0.05" />
             </geometry>
         </collision>
@@ -91,5 +91,5 @@
         <collision>
             <geometry>
-                <cylinder radius = "0.05" length= "0.04"/>
+                <sphere radius = "0.05" />
             </geometry>
         </collision>
