Commit message: Implemented slam_toolbox feature Implemented twist_mux and twist_stamper for nav2

File: description/robot_main.xacro (robot description, xacro)
@@ -21,4 +21,12 @@
     <!-- base_link -->
     <link name="base_link">
+    </link>
+    <!-- base_footprint -->
+    <joint name="base_footprint_joint" type="fixed">
+        <parent link= "base_link"/>
+        <child link= "base_footprint"/>
+        <origin xyz= "0 0 0" rpy= "0 0 0"/>
+    </joint>
+    <link name="base_footprint">
     </link>
     <!-- chasis -->
