Commit message: Implemented gazebo simulation with gz differential drive plugin
	- Created an rviz config file for simulation.
	- Created gazebo launch file.
	- Established necessary plugin configurations.
	- Created ros_gz_bridge to connect topics between ros2 and gazebo.
	- Created an template gazebo world as empty.sdf

File: description/robot.urdf.xacro (robot description, xacro)
@@ -2,3 +2,4 @@
 <robot xmlns:xacro="http://www.ros.org/wiki/xacro"  name="robot">
     <xacro:include filename = "robot_main.xacro" />
+    <xacro:include filename = "gazebo_control.xacro" />
 </robot>

File: description/robot_main.xacro (robot description, xacro)
@@ -1,4 +1,4 @@
 <?xml version="1.0"?>
-<robot xmlns:xacro="http://www.ros.org/wiki/xacro"  name="robot">
+<robot xmlns:xacro="http://www.ros.org/wiki/xacro">
     <xacro:include filename = "inertial_macros.xacro" />
     <!-- Colors -->
@@ -10,5 +10,5 @@
     </material>
     <material name= "orange">
-        <color rgba= "1 0.35 0 1"/>
+        <color rgba= "1 0.25 0 1"/>
     </material>
     <material name="cyan">
@@ -46,4 +46,7 @@
         </xacro:inertial_box>
     </link>
+    <gazebo reference="chasis">
+        <material>Gazebo/Black</material>
+    </gazebo>
     <!-- left_wheel -->
     <joint name="left_wheel_joint" type="continuous">
@@ -69,4 +72,7 @@
         </xacro:inertial_cylinder>
     </link>
+    <gazebo reference="left_wheel">
+        <material>Gazebo/Orange</material>
+    </gazebo>
     <!-- right_wheel -->
     <joint name="right_wheel_joint" type="continuous">
@@ -92,4 +98,7 @@
         </xacro:inertial_cylinder>
     </link>
+    <gazebo reference="right_wheel">
+        <material>Gazebo/Orange</material>
+    </gazebo>
     <!-- caster_wheel -->
     <joint name="caster_wheel_joint" type="fixed">
@@ -114,3 +123,8 @@
         </xacro:inertial_sphere>
     </link>
+    <gazebo reference="caster_wheel">
+        <material>Gazebo/Orange</material>
+        <mu1 value= "0.0001"/>
+        <mu2 value= "0.0001"/>
+    </gazebo>
 </robot>

Commit message: Implemented ros2_control for physical diff drive robot (no more sim). Created robot.launch.py file for physical robot control. Established hardware interface connection for the robot.
Hardware interface repo & denpendeny:
https://github.com/joshnewans/serial
https://github.com/joshnewans/diffdrive_arduino

File: description/robot.urdf.xacro (robot description, xacro)
@@ -2,4 +2,5 @@
 <robot xmlns:xacro="http://www.ros.org/wiki/xacro"  name="robot">
     <xacro:arg name="use_ros2_control"              default="true"/>
+    <xacro:arg name="use_ros2_control_gz_sim"       default="false"/>
     <!-- Robot_frames -->
     <xacro:include filename = "robot_main.xacro" />

File: description/ros2_control.xacro (robot description, xacro)
@@ -1,32 +1,64 @@
 <?xml version="1.0"?>
 <robot xmlns:xacro="http://www.ros.org/wiki/xacro">
-    <ros2_control name="minibot_ros2_control" type="system">
-        <hardware>
-            <plugin>gz_ros2_control/GazeboSimSystem</plugin>
-        </hardware>
-        <joint name="left_wheel_joint">
-            <command_interface name="velocity">
-                <param name="min">-10</param>
-                <param name="max">10</param>
-            </command_interface>
-            <state_interface name="velocity"/>
-            <state_interface name="position"/>
-        </joint>
-        <joint name="right_wheel_joint">
-            <command_interface name="velocity">
-                <param name="min">-10</param>
-                <param name="max">10</param>
-            </command_interface>
-            <state_interface name="velocity"/>
-            <state_interface name="position"/>
-        </joint>
-    </ros2_control>
-    <gazebo>
-        <plugin filename="gz_ros2_control-system"
-            name="gz_ros2_control::GazeboSimROS2ControlPlugin">
-            <parameters>
-                $(find minibot)/config/controller.yaml
-            </parameters>
-        </plugin>
-    </gazebo>
+    <xacro:unless value="$(arg use_ros2_control_gz_sim)">
+        <ros2_control name="RobotSystem" type="system">
+            <hardware>
+                <plugin>diffdrive_arduino/DiffDriveArduinoHardware</plugin>
+                    <param name="left_wheel_name">left_wheel_joint</param>
+                    <param name="right_wheel_name">right_wheel_joint</param>
+                    <param name="loop_rate">30</param>
+                    <param name="device">/dev/ttyUSB0</param>
+                    <param name="baud_rate">115200</param>
+                    <param name="timeout_ms">1000</param>
+                    <param name="enc_counts_per_rev">616</param>
+            </hardware>
+            <joint name="left_wheel_joint">
+                <command_interface name="velocity">
+                    <param name="min">-10</param>
+                    <param name="max">10</param>
+                </command_interface>
+                <state_interface name="position"/>
+                <state_interface name="velocity"/>
+            </joint>
+            <joint name="right_wheel_joint">
+                <command_interface name="velocity">
+                    <param name="min">-10</param>
+                    <param name="max">10</param>
+                </command_interface>
+                <state_interface name="position"/>
+                <state_interface name="velocity"/>
+            </joint>
+        </ros2_control>
+    </xacro:unless>
+    <xacro:if value="$(arg use_ros2_control_gz_sim)">
+        <ros2_control name="minibot_ros2_control" type="system">
+            <hardware>
+                <plugin>gz_ros2_control/GazeboSimSystem</plugin>
+            </hardware>
+            <joint name="left_wheel_joint">
+                <command_interface name="velocity">
+                    <param name="min">-10</param>
+                    <param name="max">10</param>
+                </command_interface>
+                <state_interface name="velocity"/>
+                <state_interface name="position"/>
+            </joint>
+            <joint name="right_wheel_joint">
+                <command_interface name="velocity">
+                    <param name="min">-10</param>
+                    <param name="max">10</param>
+                </command_interface>
+                <state_interface name="velocity"/>
+                <state_interface name="position"/>
+            </joint>
+        </ros2_control>
+        <gazebo>
+            <plugin filename="gz_ros2_control-system"
+                name="gz_ros2_control::GazeboSimROS2ControlPlugin">
+                <parameters>
+                    $(find minibot)/config/controller_gz_sim.yaml
+                </parameters>
+            </plugin>
+        </gazebo>
+    </xacro:if>
 </robot>
