Commit message: Updated robot URDF and related files to match the robot
	- Update robot URDF, and config files to match the robot.
	- Update sensors URDF to match the robot.
	- Rename folder "controller" to "ros2_control_demo_action"
	- Fixed CMakeLists.txt for filename change

File: description/camera.xacro (robot description, xacro)
@@ -1,14 +1,19 @@
 <?xml version="1.0"?>
 <robot xmlns:xacro="http://www.ros.org/wiki/xacro" name="robot">
+    <xacro:property name="camera_length"             value="0.01"/>
+    <xacro:property name="camera_width"              value="0.03"/>
+    <xacro:property name="camera_height"             value="0.03"/>
+    <xacro:property name="camera_offset_x"           value="0.318"/>
+    <xacro:property name="camera_offset_z"           value="0.063"/>
     <!-- Camera -->
     <joint name="camera_joint" type="fixed">
         <parent link="chasis"/>
         <child link="camera_link"/>
-        <origin xyz="0.305 0.0 0.08" rpy="0 0 0"/>
+        <origin xyz="${camera_offset_x} 0.0 ${camera_offset_z}" rpy="0 0 0"/>
     </joint>
     <link name="camera_link">
         <visual>
             <geometry>
-                <box size="0.01 0.03 0.03" />
+                <box size="${camera_length} ${camera_width} ${camera_height}" />
             </geometry>
             <material name="orange"/>

File: description/depth_camera.xacro (robot description, xacro)
@@ -1,14 +1,19 @@
 <?xml version="1.0"?>
 <robot xmlns:xacro="http://www.ros.org/wiki/xacro" name="robot">
+    <xacro:property name="RGBD_length"             value="0.01"/>
+    <xacro:property name="RGBD_width"              value="0.09"/>
+    <xacro:property name="RGBD_height"             value="0.03"/>
+    <xacro:property name="RGBD_offset_x"           value="0.318"/>
+    <xacro:property name="RGBD_offset_z"           value="0.063"/>
     <!-- RGB_Depth camera -->
     <joint name="camera_joint" type="fixed">
         <parent link="chasis"/>
         <child link="camera_link"/>
-        <origin xyz="0.305 0.0 0.08" rpy="0 0 0"/>
+        <origin xyz="${RGBD_offset_x} 0.0 ${RGBD_offset_z}" rpy="0 0 0"/>
     </joint>
     <link name="camera_link">
         <visual>
             <geometry>
-                <box size="0.01 0.09 0.03" />
+                <box size="${RGBD_length} ${RGBD_width} ${RGBD_height}" />
             </geometry>
             <material name="orange"/>

File: description/gz_diff_drive_control.xacro (robot description, xacro)
@@ -7,6 +7,6 @@
             <left_joint>left_wheel_joint</left_joint>
             <right_joint>right_wheel_joint</right_joint>
-            <wheel_separation>0.34</wheel_separation>
-            <wheel_radius>0.05</wheel_radius>
+            <wheel_separation>0.266</wheel_separation>
+            <wheel_radius>0.034</wheel_radius>
             <!-- Limits -->
             <max_wheel_torque>200</max_wheel_torque>

File: description/lidar.xacro (robot description, xacro)
@@ -1,14 +1,18 @@
 <?xml version="1.0"?>
 <robot xmlns:xacro="http://www.ros.org/wiki/xacro" name="robot">
+    <xacro:property name="lidar_radius"             value="0.025"/>
+    <xacro:property name="lidar_thickness"          value="0.040"/>
+    <xacro:property name="lidar_offset_x"           value="0.230"/>
+    <xacro:property name="lidar_offset_z"           value="0.098"/>
     <!-- Lidar -->
     <joint name="lidar_joint" type="fixed">
         <parent link="chasis"/>
         <child link="lidar_frame"/>
-        <origin xyz="0.1 0.0 0.175" rpy="0 0 0"/>
+        <origin xyz="${lidar_offset_x} 0.0 ${lidar_offset_z}" rpy="0 0 0"/>
     </joint>
     <link name="lidar_frame">
         <visual>
             <geometry>
-                <cylinder radius="0.05" length="0.04"/>
+                <cylinder radius="${lidar_radius}" length="${lidar_thickness}"/>
             </geometry>
             <material name="orange"/>
@@ -16,8 +20,8 @@
         <collision>
             <geometry>
-                <cylinder radius="0.05" length="0.04"/>
+                <cylinder radius="${lidar_radius}" length="${lidar_thickness}"/>
             </geometry>
         </collision>
-        <xacro:inertial_cylinder mass="0.1" radius="0.05" length="0.04">
+        <xacro:inertial_cylinder mass="0.1" radius="${lidar_radius}" length="${lidar_thickness}">
             <origin xyz="0 0 0" rpy="0 0 0"/>
         </xacro:inertial_cylinder>

File: description/robot_main.xacro (robot description, xacro)
@@ -2,4 +2,18 @@
 <robot xmlns:xacro="http://www.ros.org/wiki/xacro">
     <xacro:include filename = "inertial_macros.xacro" />
+    <xacro:property name="chassis_length"           value="0.320"/>
+    <xacro:property name="chassis_width"            value="0.240"/>
+    <xacro:property name="chassis_height"           value="0.078"/>
+    <xacro:property name="chassis_mass"             value="0.700"/>
+    <xacro:property name="wheel_radius"             value="0.034"/>
+    <xacro:property name="wheel_thickness"          value="0.026"/>
+    <xacro:property name="wheel_mass"               value="0.050"/>
+    <xacro:property name="wheel_offset_x"           value="0.133"/>
+    <xacro:property name="wheel_offset_y"           value="0.133"/>
+    <xacro:property name="wheel_offset_z"           value="0.020"/>
+    <xacro:property name="caster_wheel_radius"      value="${wheel_radius - wheel_offset_z}"/>
+    <xacro:property name="caster_wheel_mass"        value="0.010"/>
+    <xacro:property name="caster_wheel_offset_x"    value="0.230"/>
+    <xacro:property name="caster_wheel_offset_z"    value="${wheel_offset_z - wheel_radius + caster_wheel_radius}"/>
     <!-- Colors -->
     <material name="white">
@@ -34,22 +48,22 @@
         <parent link= "base_link"/>
         <child link= "chasis"/>
-        <origin xyz= "-0.1 0 0"/>
+        <origin xyz= "${-wheel_offset_x} 0 ${-wheel_offset_z}"/>
     </joint>
     <link name="chasis">
         <visual>
-            <origin xyz= "0.15 0 0.075" rpy= "0 0 0"/>
+            <origin xyz= "${chassis_length/2} 0 ${chassis_height/2}" rpy= "0 0 0"/>
             <geometry>
-                <box size = "0.3 0.3 0.15"/>
+                <box size = "${chassis_length} ${chassis_width} ${chassis_height}"/>
             </geometry>
             <material name= "black"/>
         </visual>
         <collision>
-            <origin xyz= "0.15 0 0.075" rpy= "0 0 0"/>
+            <origin xyz= "${chassis_length/2} 0 ${chassis_height/2}" rpy= "0 0 0"/>
             <geometry>
-                <box size = "0.3 0.3 0.15"/>
+                <box size = "${chassis_length} ${chassis_width} ${chassis_height}"/>
             </geometry>
         </collision>
-        <xacro:inertial_box mass= "0.5" x="0.3" y="0.3" z="0.15">
-            <origin xyz= "0.15 0 0.075" rpy= "0 0 0"/>
+        <xacro:inertial_box mass= "0.5" x="${chassis_length}" y="${chassis_width}" z="${chassis_height}">
+            <origin xyz= "${chassis_length/2} 0 ${chassis_height/2}" rpy= "0 0 0"/>
         </xacro:inertial_box>
     </link>
@@ -61,5 +75,5 @@
         <parent link= "base_link"/>
         <child link= "left_wheel"/>
-        <origin xyz= "0 0.17 0" rpy = "${pi/2} 0 0"/>
+        <origin xyz= "0 ${wheel_offset_y} 0" rpy = "${pi/2} 0 0"/>
         <axis xyz= "0 0 -1"/>
     </joint>
@@ -67,5 +81,5 @@
         <visual>
             <geometry>
-                <cylinder radius = "0.05" length= "0.04"/>
+                <cylinder radius = "${wheel_radius}" length= "${wheel_thickness}"/>
             </geometry>
             <material name= "orange"/>
@@ -73,8 +87,8 @@
         <collision>
             <geometry>
-                <sphere radius = "0.05" />
+                <sphere radius = "${wheel_radius}" />
             </geometry>
         </collision>
-        <xacro:inertial_cylinder mass = "0.1" radius= "0.05" length= "0.04">
+        <xacro:inertial_cylinder mass = "${wheel_mass}" radius= "${wheel_radius}" length= "${wheel_thickness}">
             <origin xyz= "0 0 0" rpy= "0 0 0"/>
         </xacro:inertial_cylinder>
@@ -87,5 +101,5 @@
         <parent link= "base_link"/>
         <child link= "right_wheel"/>
-        <origin xyz= "0 -0.17 0" rpy = "${pi/2} 0 0"/>
+        <origin xyz= "0 ${-wheel_offset_y} 0" rpy = "${pi/2} 0 0"/>
         <axis xyz= "0 0 -1"/>
     </joint>
@@ -93,5 +107,5 @@
         <visual>
             <geometry>
-                <cylinder radius = "0.05" length= "0.04"/>
+                <cylinder radius = "${wheel_radius}" length= "${wheel_thickness}"/>
             </geometry>
             <material name= "orange"/>
@@ -99,8 +113,8 @@
         <collision>
             <geometry>
-                <sphere radius = "0.05" />
+                <sphere radius = "${wheel_radius}" />
             </geometry>
         </collision>
-        <xacro:inertial_cylinder mass= "0.1" radius= "0.05" length= "0.04">
+        <xacro:inertial_cylinder mass = "${wheel_mass}" radius= "${wheel_radius}" length= "${wheel_thickness}">
             <origin xyz= "0 0 0" rpy= "0 0 0"/>
         </xacro:inertial_cylinder>
@@ -113,10 +127,10 @@
         <parent link= "chasis"/>
         <child link= "caster_wheel"/>
-        <origin xyz= "0.24 0 0"/>
+        <origin xyz= "${caster_wheel_offset_x} 0 0"/>
     </joint>
     <link name="caster_wheel">
         <visual>
             <geometry>
-                <sphere radius = "0.05"/>
+                <sphere radius = "${caster_wheel_radius}"/>
             </geometry>
             <material name= "orange"/>
@@ -124,8 +138,8 @@
         <collision>
             <geometry>
-                <sphere radius = "0.05"/>
+                <sphere radius = "${caster_wheel_radius}"/>
             </geometry>
         </collision>
-        <xacro:inertial_sphere mass= "0.1" radius= "0.05">
+        <xacro:inertial_sphere mass= "${caster_wheel_mass}" radius= "${caster_wheel_radius}">
             <origin xyz= "0 0 0" rpy= "0 0 0"/>
         </xacro:inertial_sphere>
