Commit message: Configured parameters and to match the robot and consolidated the launch files.
	- Created an rviz config file for testing the robot.
	- Included joystick teleop, slam_toolbox and nav2 stack implementation into a launch file seperately for both simulation and physical robot.
	- Configured some parameters to fit the testing environment.

File: description/lidar.xacro (robot description, xacro)
@@ -9,5 +9,5 @@
         <parent link="chasis"/>
         <child link="lidar_frame"/>
-        <origin xyz="${lidar_offset_x} 0.0 ${lidar_offset_z}" rpy="0 0 0"/>
+        <origin xyz="${lidar_offset_x} 0.0 ${lidar_offset_z}" rpy="0 0 ${pi}"/>
     </joint>
     <link name="lidar_frame">
